File: brd/BeagleCap.brd (EAGLE design)
At the start: 140 x 177.5 mm, 20 parts, among them CN1 DS18B20, IC2 7805TV, U1 DHT22, X1 Conn BNC : pH, X2 Conn BNC : Dissolved Oxygen, X3 Conn BNC : Conductivity

Commit message: Schematic updated with new PCB
Done by JayMcGee
Parts:
- removed BATT: (no value), con-wago-500:W237-102
- removed CN1: DS18B20, adafruit:JSTPH3
- added D1, D2: 1N4007, diode:DO41-10
- added D3, D4: 1N4148DO35-10, diode:DO35-10
- added J2: DS18B20, con-amp:10X03MTA
- added J3: Battery, con-amp:10X03MTA
- added J4: (no value), con-amp:10X05MTA
- added KK1: SK104-PAD, heatsink:SK104-PAD
- added LED1: (no value), led:LED5MM
- added R10, R9: 4.7K, adafruit:0207/10
- added R7: 330, adafruit:0207/10
- added R8: 1K, adafruit:0207/10
- added U$5: ATLAS_STAMP, LEDscape:ATLAS_STAMP
- added X4: Conn BNC : ORP, con-coax:AMP_227161
- C1: value 0.33uF -> 1uF; device adafruit:C050-024X044 -> rcl:E2-5
- C2: value 0.1uf -> 10uF; device adafruit:C050-024X044 -> rcl:E2-5
- moved U$1 177.8 mm to (-93.4, 22.1), flipped to the bottom
- moved BARREL 173.2 mm to (-72.5, 83.0), turned to 270 degrees
- moved R5 107.9 mm to (-35.0, 11.5)
- moved R6 107.9 mm to (-35.0, 7.00)
- moved C1 94.4 mm to (-8.50, 82.0), turned to 270 degrees
- moved IC2 88.3 mm to (14.4, 81.3), flipped to the bottom, turned to 0 degrees
- moved C2 73.6 mm to (38.0, 81.5), turned to 270 degrees
- moved X2 50.0 mm to (-72.0, 9.50), flipped to the top, turned to 90 degrees
- moved X3 48.3 mm to (-72.0, -33.0), flipped to the top, turned to 90 degrees
- moved U$3 44.5 mm to (-63.0, 16.5), turned to 270 degrees
- moved X1 41.1 mm to (-72.0, -11.5), flipped to the top, turned to 90 degrees
- moved U1 38.0 mm to (-8.89, -7.76)
- moved R4 36.5 mm to (-23.6, 7.16)
- moved R1 35.6 mm to (-12.8, 7.16)
- moved U$4 32.1 mm to (-63.0, -26.0), turned to 270 degrees
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Connections:
- removed net VCC: CN1.1, R2.2, R4.1, R5.2, R6.2, U$1.50, U$2.VCC, U$3.VCC, U$4.VCC, U1.VDD
- new net 3.3V: J2.3, R2.2, R4.1, R5.2, R6.2, U$1.50, U$2.VCC, U$3.VCC, U$4.VCC, U$5.VCC, U1.VDD
- new net N$1: D1.A, D2.A, J3.3
- new net N$10: J4.3, R8.1
- new net N$11: D4.C, J4.4, R10.2
- new net N$2: LED1.K, R7.2
- new net N$9: D3.C, J4.2, R9.2
- new net ORP_SENSOR: U$5.PRB, X4.1
- new net P: D4.A, U$1.88
- new net RX: R8.2, U$1.72
- new net TX: D3.A, U$1.70
- net 5V: now also C2.+, J4.1, LED1.A, R10.1, R9.1; no longer C2.1
- net GND: now also C1.-, C2.-, J2.2, J3.2, J4.5, KK1.K1, KK1.K2, R7.1, U$5.GND, U$5.PGND, X4.2; no longer BATT.2, C1.2, C2.2, CN1.2
- net I2C2_SCL: now also U$5.TX
- net I2C2_SDA: now also U$5.RX
- net N$5: now also J2.1; no longer CN1.3
- net VIN: now also C1.+, D1.C, D2.C; no longer BATT.1, C1.1
Routing:
- net GND: track 17.6 -> 376.9 mm
- net 5V: track 7.03 -> 284.3 mm
- net 3.3V: track 0.00 -> 259.7 mm
- net TX: track 0.00 -> 148.2 mm
- net RX: track 0.00 -> 143.7 mm
- net P: track 0.00 -> 134.1 mm
- net I2C2_SCL: track 0.00 -> 82.2 mm
- net I2C2_SDA: track 0.00 -> 80.8 mm
- net VIN: track 7.09 -> 65.3 mm
- net N$9: track 0.00 -> 29.0 mm
- net N$11: track 0.00 -> 29.0 mm
- net N$1: track 0.00 -> 20.9 mm
- net N$5: track 19.1 -> 0.00 mm
- net N$10: track 0.00 -> 11.4 mm
- net N$2: track 0.00 -> 6.13 mm
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Other:
- board size 140 x 177.5 mm -> 152.5 x 152 mm
- board text added: "AQUARIUS"
- board text added: "Jean-Philippe Fournier Jean-Pascal McGee"
- board text added: "SIM908"
