File: brd/Jp_brd/Aquarius.brd (EAGLE design)
At the start: 75.7 x 129 mm, 40 parts, among them IC1 74123D, J2 DS18B20, J4 GSM/GPS, U1 DHT22, U2 DS3231SN, X1 Conn BNC : pH, X2 Conn BNC : Dissolved Oxygen, X3 Conn BNC : Conductivity, X4 Batt.1, X5 Batt.2

Commit message: Mise a jour du PCB version Jay_brd pour finalisation
Parts:
- added Q1, Q2, Q3, Q4: BSS138, m-pad-2.1:SOT23
- L1: device resistor:0204/7 -> rcl:LAL04
- moved L1 6.49 mm to (7.87, 23.6), turned to 90 degrees
Routing:
- net N$16: track 24.6 -> 12.3 mm
- net N$13: track 34.6 -> 38.1 mm
Changed lines of the file:
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@@
 <text x="37.1094" y="1.2192" size="1.778" layer="25">Lab</text>
 <text x="-2.2098" y="-50.2158" size="1.778" layer="25" rot="R180">Temp.</text>
-<text x="22.7838" y="-7.0104" size="1.778" layer="25">LM2678</text>
+<text x="32.0802" y="14.3256" size="1.778" layer="25" rot="R270">LM2678</text>
 <text x="149.9024" y="36.466" size="1.778" layer="144">LAYER-STACK</text>
 <text x="-79.8914" y="-70.6331" size="1.778" layer="145">01-16</text>
@@
 </element>
 <element name="C3" library="resistor" package="E2,5-6E" value="4.7uF" x="14.4902" y="33.4946" smashed="yes">
-<attribute name="NAME" x="17.1112" y="35.2504" size="1.27" layer="25" rot="R90"/>
+<attribute name="NAME" x="11.9296" y="35.098" size="1.27" layer="25" rot="R90"/>
 <attribute name="VALUE" x="21.0688" y="30.0148" size="1.27" layer="27" rot="R90"/>
 </element>
 <element name="C5" library="rcl" package="C0805" value="100nF" x="24.1432" y="33.1908" smashed="yes">
-<attribute name="NAME" x="21.9272" y="32.0172" size="1.27" layer="25" rot="R90"/>
+<attribute name="NAME" x="24.2894" y="34.3032" size="1.27" layer="25" rot="R90"/>
 <attribute name="VALUE" x="27.566" y="30.9504" size="1.27" layer="27" rot="R90"/>
 </element>
 <element name="C6" library="rcl" package="C0805" value="10nF" x="14.425" y="26.3016" smashed="yes" rot="R180">
-<attribute name="NAME" x="9.6034" y="26.1748" size="1.27" layer="25"/>
+<attribute name="NAME" x="12.4228" y="23.965" size="1.27" layer="25"/>
 <attribute name="VALUE" x="12.3422" y="25.8698" size="1.27" layer="27" rot="R180"/>
 </element>
@@
 </element>
 <element name="C1" library="resistor" package="E2,5-6E" value="180uF" x="7.175" y="36.1438" smashed="yes">
-<attribute name="NAME" x="13.6822" y="38.433" size="1.27" layer="25" rot="R90"/>
+<attribute name="NAME" x="4.6906" y="37.3662" size="1.27" layer="25" rot="R90"/>
 <attribute name="VALUE" x="13.7536" y="32.664" size="1.27" layer="27" rot="R90"/>
 </element>
-<element name="L1" library="resistor" package="0204/7" value="22uH" x="10.507" y="17.6272" smashed="yes" rot="R180">
-<attribute name="NAME" x="9.9572" y="21.7338" size="1.27" layer="25" rot="R270"/>
-<attribute name="VALUE" x="9.9056" y="19.6428" size="1.27" layer="27" rot="R90"/>
+<element name="L1" library="rcl" package="LAL04" value="22uH" x="7.8736" y="23.5544" smashed="yes" rot="R90">
+<attribute name="NAME" x="7.1034" y="18.0082" size="1.27" layer="25" rot="R180"/>
+<attribute name="VALUE" x="9.8892" y="24.1558" size="1.27" layer="27"/>
 </element>
 <element name="X4" library="con-weidmueller-sl35" package="180G-2" value="Batt.1" x="23.9268" y="63.0174" smashed="yes" rot="R180">
@@
 <element name="DRILEGEND" library="drilegend" package="DRILEGEND" value="" x="-40.52140625" y="-64.88000625"/>
 <element name="D4" library="diode" package="DO201T15" value="" x="1.524" y="26.5176" smashed="yes" rot="R90">
-<attribute name="NAME" x="5.0038" y="33.6296" size="1.27" layer="25" ratio="10" rot="R180"/>
+<attribute name="NAME" x="2.4892" y="24.3332" size="1.27" layer="25" ratio="10" rot="R180"/>
 <attribute name="VALUE" x="3.683" y="23.9776" size="1.27" layer="27" ratio="10" rot="R90"/>
 </element>
@@
 <element name="R8" library="adafruit" package="R0805" value="4.7K" x="27.5844" y="-49.6062"/>
 <element name="R9" library="adafruit" package="R0805" value="4.7K" x="27.5844" y="-52.8828"/>
+<element name="Q2" library="m-pad-2.1" package="SOT23" value="BSS138" x="-78.0288" y="-102.1842"/>
+<element name="Q3" library="m-pad-2.1" package="SOT23" value="BSS138" x="-78.0288" y="-109.4994"/>
+<element name="Q4" library="m-pad-2.1" package="SOT23" value="BSS138" x="-78.0288" y="-116.8146"/>
+<element name="Q1" library="m-pad-2.1" package="SOT23" value="BSS138" x="-78.0288" y="-124.1298"/>
 </elements>
 <signals>
@@
 <contactref element="C6" pad="2"/>
 <contactref element="L1" pad="1"/>
-<wire x1="13.475" y1="26.3016" x2="13.2714" y2="26.3016" width="1.27" layer="1"/>
-<wire x1="13.2714" y1="26.3016" x2="11.5062" y2="24.5364" width="1.27" layer="1"/>
-<wire x1="11.5062" y1="24.5364" x2="11.5062" y2="21.8694" width="1.27" layer="1"/>
-<wire x1="11.5062" y1="21.8694" x2="14.1732" y2="19.2024" width="1.27" layer="1"/>
-<wire x1="14.1732" y1="19.2024" x2="14.1732" y2="17.771" width="1.27" layer="1"/>
-<wire x1="14.1732" y1="17.771" x2="14.317" y2="17.6272" width="1.27" layer="1"/>
-<wire x1="19.4586" y1="27.4246" x2="17.4572" y2="27.4246" width="1.016" layer="1"/>
-<wire x1="17.4572" y1="27.4246" x2="16.764" y2="28.1178" width="1.016" layer="1"/>
-<wire x1="16.764" y1="28.1178" x2="13.8684" y2="28.1178" width="1.016" layer="1"/>
-<wire x1="13.8684" y1="28.1178" x2="13.5636" y2="27.813" width="1.016" layer="1"/>
-<wire x1="13.5636" y1="27.813" x2="13.5636" y2="26.3902" width="1.016" layer="1"/>
-<wire x1="13.5636" y1="26.3902" x2="13.475" y2="26.3016" width="1.016" layer="1"/>
-<wire x1="19.4586" y1="27.4246" x2="19.4586" y2="31.5192" width="1.016" layer="1"/>
-<wire x1="19.4586" y1="31.5192" x2="19.431" y2="31.5468" width="1.016" layer="1"/>
-<via x="19.431" y="31.5468" extent="1-16" drill="0.6"/>
-<wire x1="19.431" y1="31.5468" x2="19.431" y2="35.7236" width="1.016" layer="16"/>
-<wire x1="19.431" y1="35.7236" x2="24.816" y2="41.1086" width="1.016" layer="16"/>
+<wire x1="13.475" y1="26.3016" x2="13.475" y2="27.8768" width="1.016" layer="1"/>
+<wire x1="13.475" y1="27.8768" x2="14.4018" y2="28.8036" width="1.016" layer="1"/>
+<wire x1="14.4018" y1="28.8036" x2="18.0796" y2="28.8036" width="1.016" layer="1"/>
+<wire x1="18.0796" y1="28.8036" x2="19.4586" y2="27.4246" width="1.016" layer="1"/>
+<wire x1="24.816" y1="41.1086" x2="24.7256" y2="41.1086" width="1.016" layer="16"/>
+<wire x1="24.7256" y1="41.1086" x2="19.3548" y2="35.7378" width="1.016" layer="16"/>
+<wire x1="19.3548" y1="35.7378" x2="19.3548" y2="30.7086" width="1.016" layer="16"/>
+<wire x1="19.3548" y1="30.7086" x2="19.431" y2="30.6324" width="1.016" layer="16"/>
+<via x="19.431" y="30.6324" extent="1-16" drill="0.6" shape="square"/>
+<wire x1="19.431" y1="30.6324" x2="19.431" y2="30.155" width="1.016" layer="1"/>
+<wire x1="19.431" y1="30.155" x2="18.0796" y2="28.8036" width="1.016" layer="1"/>
+<wire x1="13.475" y1="26.3016" x2="13.475" y2="18.047" width="1.27" layer="1"/>
+<wire x1="13.475" y1="18.047" x2="12.4206" y2="16.9926" width="1.27" layer="1"/>
+<wire x1="12.4206" y1="16.9926" x2="8.0854" y2="16.9926" width="1.27" layer="1"/>
+<wire x1="8.0854" y1="16.9926" x2="7.8736" y2="17.2044" width="1.27" layer="1"/>
 </signal>
 <signal name="N$9">
 <contactref element="LM2678" pad="3"/>
 <contactref element="C6" pad="1"/>
-<wire x1="15.375" y1="26.3016" x2="15.9132" y2="26.3016" width="0.8128" layer="1"/>
-<wire x1="15.9132" y1="26.3016" x2="17.2974" y2="24.9174" width="0.8128" layer="1"/>
-<wire x1="17.2974" y1="24.9174" x2="19.4458" y2="24.9174" width="0.8128" layer="1"/>
-<wire x1="19.4458" y1="24.9174" x2="19.4586" y2="24.9046" width="0.8128" layer="1"/>
+<wire x1="19.4586" y1="24.9046" x2="16.772" y2="24.9046" width="1.27" layer="1"/>
+<wire x1="16.772" y1="24.9046" x2="15.375" y2="26.3016" width="1.27" layer="1"/>
 </signal>
 <signal name="N$11">
@@
 <contactref element="D4" pad="A"/>
 <contactref element="C1" pad="+"/>
-<wire x1="1.524" y1="34.1376" x2="1.524" y2="28.7274" width="1.27" layer="1"/>
-<wire x1="1.524" y1="28.7274" x2="6.7818" y2="23.4696" width="1.27" layer="1"/>
-<wire x1="6.7818" y1="23.4696" x2="6.7818" y2="17.712" width="1.27" layer="1"/>
-<wire x1="6.7818" y1="17.712" x2="6.697" y2="17.6272" width="1.27" layer="1"/>
-<wire x1="1.524" y1="34.1376" x2="1.524" y2="35.3568" width="1.016" layer="1"/>
-<wire x1="1.524" y1="35.3568" x2="1.9812" y2="35.814" width="1.016" layer="1"/>
-<wire x1="1.9812" y1="35.814" x2="5.5752" y2="35.814" width="1.016" layer="1"/>
-<wire x1="5.5752" y1="35.814" x2="5.905" y2="36.1438" width="1.016" layer="1"/>
+<wire x1="5.905" y1="36.1438" x2="3.5302" y2="36.1438" width="1.27" layer="1"/>
+<wire x1="3.5302" y1="36.1438" x2="1.524" y2="34.1376" width="1.27" layer="1"/>
+<wire x1="7.8736" y1="29.9044" x2="7.8736" y2="31.8266" width="1.27" layer="1"/>
+<wire x1="7.8736" y1="31.8266" x2="6.2484" y2="33.4518" width="1.27" layer="1"/>
+<wire x1="6.2484" y1="33.4518" x2="6.2484" y2="35.8004" width="1.27" layer="1"/>
+<wire x1="6.2484" y1="35.8004" x2="5.905" y2="36.1438" width="1.27" layer="1"/>
 </signal>
 <signal name="N$18">
