File: brd/Jp_brd/Aquarius.sch (EAGLE design)
At the start: 39 parts, among them IC1 74123D, J2 DS18B20, J4 GSM/GPS, U1 DHT22, U2 DS3231SN, X1 Conn BNC : pH, X2 Conn BNC : Dissolved Oxygen, X3 Conn BNC : Conductivity, X4 Batt.1, X5 Batt.2

Commit message: Mise a jour du PCB version Jay_brd pour finalisation
Parts:
- added Q1, Q2, Q3, Q4: BSS138, m-pad-2.1:BSS138
- L1: device resistor:L-US0204/7 -> rcl:L-USLAL04
Changed lines of the file:
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@@
 <part name="D3" library="diode" deviceset="SCHOTTKY-DIODE" device="DO201T15" value="3A"/>
 <part name="C1" library="resistor" deviceset="CPOL-US" device="E2,5-6E" value="180uF"/>
-<part name="L1" library="resistor" deviceset="L-US" device="0204/7" value="22uH"/>
+<part name="L1" library="rcl" deviceset="L-US" device="LAL04" value="22uH"/>
 <part name="SUPPLY4" library="supply2" deviceset="VCC" device=""/>
 <part name="SUPPLY10" library="supply2" deviceset="VCC" device=""/>
@@
 <part name="R9" library="adafruit" deviceset="R-US_" device="R0805" value="4.7K"/>
 <part name="SUPPLY7" library="supply2" deviceset="GND" device=""/>
+<part name="Q2" library="m-pad-2.1" deviceset="BSS138" device=""/>
+<part name="Q3" library="m-pad-2.1" deviceset="BSS138" device=""/>
+<part name="Q4" library="m-pad-2.1" deviceset="BSS138" device=""/>
+<part name="Q1" library="m-pad-2.1" deviceset="BSS138" device=""/>
 </parts>
 <sheets>
@@
 <instance part="R9" gate="G$1" x="167.64" y="81.28" rot="R90"/>
 <instance part="SUPPLY7" gate="GND" x="218.44" y="45.72"/>
+<instance part="Q2" gate="G$1" x="86.36" y="-55.88" rot="R270"/>
+<instance part="Q3" gate="G$1" x="96.52" y="-71.12" rot="R270"/>
+<instance part="Q4" gate="G$1" x="119.38" y="-71.12" rot="R270"/>
+<instance part="Q1" gate="G$1" x="73.66" y="-71.12" rot="R270"/>
 </instances>
 <busses>
