File: brd/Jay_brd/Aquarius.brd (EAGLE design)
At the start: 107.1 x 98.9 mm, 40 parts, among them IC1 74123D, J2 DS18B20, J4 GSM/GPS, SW2 Modes, U1 DHT22, U2 DS3231SN, X1 Conn BNC : pH, X2 Conn BNC : Dissolved Oxygen, X3 Conn BNC : Conductivity, X4 Batt.1, X5 Batt.2

Commit message: Mise a jour du PCB version Jay_brd pour finalisation
Parts:
- removed DRILEGEND: (no value), drilegend:DRILEGEND
- added JP1: (no value), jumper:JP2
- added JP2: (no value), pinhead:1X02
- added LED1: (no value), led:CHIP-LED0805
- added Q1, Q2, Q3: BSS138, m-pad-2.1:SOT23
- added R10, R12, R13, R16, R17, R18: 10K, adafruit:R0805
- added R19: 200, adafruit:R0805
- C1: device rcl:140CLH-0810 -> rcl:PANASONIC_D
- C3: device rcl:140CLH-0810 -> rcl:PANASONIC_B
- C4: device rcl:153CLV-0405 -> rcl:PANASONIC_B
- L1: device rcl:L8530M -> jt-inductors:EPCOS-10X10
- moved S1 99.3 mm to (-46.4, 33.9), turned to 180 degrees
- moved SW2 76.5 mm to (-32.1, 29.6), turned to 180 degrees
- moved C4 36.7 mm to (27.6, 45.1), turned to 270 degrees
- moved R11 34.6 mm to (-16.5, -10.9), turned to 0 degrees
- moved LM2678 30.8 mm to (-46.6, 63.3), turned to 90 degrees
- moved C6 30.3 mm to (-32.8, 55.8)
- moved D3 27.1 mm to (-25.3, 66.3)
- moved D4 27.1 mm to (-25.3, 60.0)
- moved L1 24.7 mm to (-25.1, 50.8), turned to 0 degrees
- moved R14 23.6 mm to (15.8, 21.5), turned to 270 degrees
- moved D2 22.8 mm to (0.72, 66.3)
- moved D1 22.8 mm to (0.80, 60.0)
- moved X5 22.3 mm to (15.8, 63.5), turned to 180 degrees
- moved R15 22.1 mm to (16.4, 1.43), turned to 90 degrees
- moved R6 22.1 mm to (-35.2, -4.72), turned to 180 degrees
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Connections:
- new net N$1: J4.4, Q3.3, R18.1
- new net N$22: J4.3, Q2.3, R16.1
- new net N$23: J4.2, Q1.3, R12.1
- new net N$25: JP1.2, R12.2, R16.2, R18.2
- new net N$26: LED1.A, R19.1
- new net N$27: R19.2, U$1.61
- net 5V: now also JP1.3
- net GND: now also LED1.C
- net I2C2_SCL: now also JP2.1
- net I2C2_SDA: now also JP2.2
- net N$13: now also L1.P$1; no longer L1.1
- net N$16: now also L1.P$2; no longer L1.2
- net P: now also Q3.2, R17.1; no longer J4.4
- net RX: now also Q2.2, R13.1; no longer J4.3
- net TX: now also Q1.2, R10.1; no longer J4.2
- net VCC: now also JP1.1, Q1.1, Q2.1, Q3.1, R10.2, R13.2, R17.2
Routing:
- net N$23: track 0.00 -> 105.6 mm, vias 0 -> 2
- net 5V: track 209.9 -> 311.0 mm, vias 2 -> 5
- net N$1: track 0.00 -> 90.7 mm
- net N$21: track 19.2 -> 106.1 mm, vias 0 -> 3
- net N$22: track 0.00 -> 81.7 mm
- net N$27: track 0.00 -> 70.3 mm, vias 0 -> 2
- net N$17: track 107.3 -> 37.3 mm
- net VCC: track 226.3 -> 294.7 mm, vias 1 -> 9
- net N$25: track 0.00 -> 65.9 mm, vias 0 -> 2
- net N$19: track 31.5 -> 92.4 mm, vias 0 -> 4
- net TX: track 69.1 -> 13.6 mm
- net RX: track 68.5 -> 18.6 mm
- net INT: track 73.3 -> 108.4 mm, vias 1 -> 3
- net P: track 66.2 -> 34.5 mm, vias 0 -> 1
- net N$16: track 15.0 -> 45.5 mm
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- added copper zone on layer 1, net N$28
- removed copper zone on layer 1, net GND
Other:
- board size 107.1 x 98.9 mm -> 92.7 x 99.2 mm
- board text removed: "LAYER-STACK"

Commit message: Finalisation du pcb avant le test 4pcb
Parts:
- added DRILEGEND: (no value), drilegend:DRILEGEND
- JP2: value (none) -> I2C
- moved R6 7.55 mm to (-42.6, -5.97)
- moved R5 7.51 mm to (-42.7, -2.50)
Routing:
- net VCC: track 294.7 -> 279.0 mm
- net I2C2_SCL: track 110.6 -> 117.8 mm
- net I2C2_SDA: track 124.9 -> 129.8 mm
- added copper zone on layer 1, net GND
- removed copper zone on layer 1, net N$28
Other:
- board text added: "LAYER-STACK"
- board text removed: "Temp."

Commit message: Final modifications to PCB for production
Routing:
- net GND: track 75.9 -> 84.4 mm, vias 5 -> 6
- net I2C2_SDA: track 129.8 -> 131.7 mm
Changed lines of the file:
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@@
 <layer number="27" name="tValues" color="7" fill="1" visible="yes" active="yes"/>
 <layer number="28" name="bValues" color="7" fill="1" visible="yes" active="yes"/>
-<layer number="29" name="tStop" color="7" fill="3" visible="yes" active="yes"/>
+<layer number="29" name="tStop" color="7" fill="3" visible="no" active="yes"/>
 <layer number="30" name="bStop" color="7" fill="6" visible="no" active="yes"/>
 <layer number="31" name="tCream" color="7" fill="4" visible="no" active="yes"/>
@@
 <text x="-49.53" y="37.4904" size="0.8128" layer="25">On/Off</text>
 <hole x="21.7932" y="-25.4508" drill="2.8"/>
-<hole x="21.5646" y="57.15" drill="2.8"/>
+<hole x="7.3152" y="50.5206" drill="2.8"/>
 <hole x="-59.817" y="67.9704" drill="2.8"/>
-<hole x="-42.5196" y="-20.193" drill="2.8"/>
+<hole x="-42.5958" y="-14.5542" drill="2.8"/>
 <wire x1="-11.811" y1="-28.575" x2="-11.811" y2="-27.9654" width="0.3048" layer="20"/>
 <wire x1="-11.811" y1="-27.9654" x2="-6.1722" y2="-22.3266" width="0.3048" layer="20" curve="-90"/>
@@
 <wire x1="21.7932" y1="-25.4508" x2="21.2852" y2="-24.9428" width="0.1016" layer="146"/>
 <wire x1="21.7932" y1="-25.4508" x2="21.7932" y2="-25.9588" width="0.1016" layer="146"/>
-<wire x1="21.0566" y1="57.658" x2="22.0726" y2="57.658" width="0.1016" layer="146"/>
-<wire x1="22.0726" y1="57.658" x2="21.5646" y2="57.15" width="0.1016" layer="146"/>
-<wire x1="21.5646" y1="57.15" x2="21.0566" y2="57.658" width="0.1016" layer="146"/>
-<wire x1="21.5646" y1="57.15" x2="21.5646" y2="56.642" width="0.1016" layer="146"/>
+<wire x1="6.8072" y1="51.0286" x2="7.8232" y2="51.0286" width="0.1016" layer="146"/>
+<wire x1="7.8232" y1="51.0286" x2="7.3152" y2="50.5206" width="0.1016" layer="146"/>
+<wire x1="7.3152" y1="50.5206" x2="6.8072" y2="51.0286" width="0.1016" layer="146"/>
+<wire x1="7.3152" y1="50.5206" x2="7.3152" y2="50.0126" width="0.1016" layer="146"/>
 <wire x1="-60.325" y1="68.4784" x2="-59.309" y2="68.4784" width="0.1016" layer="146"/>
 <wire x1="-59.309" y1="68.4784" x2="-59.817" y2="67.9704" width="0.1016" layer="146"/>
 <wire x1="-59.817" y1="67.9704" x2="-60.325" y2="68.4784" width="0.1016" layer="146"/>
 <wire x1="-59.817" y1="67.9704" x2="-59.817" y2="67.4624" width="0.1016" layer="146"/>
-<wire x1="-43.0276" y1="-19.685" x2="-42.0116" y2="-19.685" width="0.1016" layer="146"/>
-<wire x1="-42.0116" y1="-19.685" x2="-42.5196" y2="-20.193" width="0.1016" layer="146"/>
-<wire x1="-42.5196" y1="-20.193" x2="-43.0276" y2="-19.685" width="0.1016" layer="146"/>
-<wire x1="-42.5196" y1="-20.193" x2="-42.5196" y2="-20.701" width="0.1016" layer="146"/>
+<wire x1="-43.1038" y1="-14.0462" x2="-42.0878" y2="-14.0462" width="0.1016" layer="146"/>
+<wire x1="-42.0878" y1="-14.0462" x2="-42.5958" y2="-14.5542" width="0.1016" layer="146"/>
+<wire x1="-42.5958" y1="-14.5542" x2="-43.1038" y2="-14.0462" width="0.1016" layer="146"/>
+<wire x1="-42.5958" y1="-14.5542" x2="-42.5958" y2="-15.0622" width="0.1016" layer="146"/>
 </plain>
 <attributes>
@@
 <param name="srMinRoundness" value="0mil"/>
 <param name="srMaxRoundness" value="0mil"/>
-<param name="slThermalIsolate" value="10mil"/>
+<param name="slThermalIsolate" value="12mil"/>
 <param name="slThermalsForVias" value="0"/>
 <param name="dpMaxLengthDifference" value="10mm"/>
@@
 <attribute name="NAME" x="23.5484" y="58.9188" size="0.8128" layer="25"/>
 <attribute name="VALUE" x="26.1392" y="58.9762" size="0.8128" layer="27"/>
+<attribute name="OC_NEWARK" value="unknown" x="25.0698" y="63.4746" size="1.778" layer="27" rot="R180" display="off"/>
+<attribute name="MPN" value="" x="25.0698" y="63.4746" size="1.778" layer="27" rot="R180" display="off"/>
+<attribute name="MF" value="" x="25.0698" y="63.4746" size="1.778" layer="27" rot="R180" display="off"/>
+<attribute name="OC_FARNELL" value="unknown" x="25.0698" y="63.4746" size="1.778" layer="27" rot="R180" display="off"/>
 </element>
 <element name="X5" library="con-weidmueller-sl35" package="180G-2" value="Batt.2" x="15.7734" y="63.4746" smashed="yes" rot="R180">
 <attribute name="NAME" x="12.8042" y="58.995" size="0.8128" layer="25"/>
 <attribute name="VALUE" x="16.4618" y="58.9762" size="0.8128" layer="27"/>
+<attribute name="OC_NEWARK" value="unknown" x="15.7734" y="63.4746" size="1.778" layer="27" rot="R180" display="off"/>
+<attribute name="MPN" value="" x="15.7734" y="63.4746" size="1.778" layer="27" rot="R180" display="off"/>
+<attribute name="MF" value="" x="15.7734" y="63.4746" size="1.778" layer="27" rot="R180" display="off"/>
+<attribute name="OC_FARNELL" value="unknown" x="15.7734" y="63.4746" size="1.778" layer="27" rot="R180" display="off"/>
 </element>
 <element name="D4" library="diode" package="DO201T15" value="" x="-25.2984" y="59.9694" smashed="yes">
@@
 <vertex x="-43.2816" y="69.4944"/>
 </polygon>
-<wire x1="-29.0852" y1="-0.279" x2="-29.1614" y2="16.6894" width="0" layer="19" extent="1-1"/>
+<wire x1="-29.0852" y1="-0.279" x2="-26.5938" y2="2.2124" width="1.016" layer="1"/>
+<wire x1="-26.5938" y1="2.2124" x2="-26.5938" y2="5.4864" width="1.016" layer="1"/>
+<via x="-26.5938" y="5.4864" extent="1-16" drill="0.6" shape="square"/>
+<wire x1="-26.5938" y1="5.4864" x2="-26.5938" y2="7.1628" width="1.016" layer="16"/>
 </signal>
 <signal name="N$3">
@@
 <wire x1="-54.3306" y1="26.1366" x2="-56.4134" y2="26.1366" width="0.6096" layer="16"/>
 <wire x1="-56.4134" y1="26.1366" x2="-56.6928" y2="26.1874" width="0.6096" layer="16"/>
-<wire x1="-41.6278" y1="-5.969" x2="-40.6654" y2="-7.1628" width="0.8128" layer="1"/>
-<wire x1="-40.6654" y1="-7.1628" x2="-40.6654" y2="-15.494" width="0.8128" layer="1"/>
-<wire x1="-40.6654" y1="-15.494" x2="-35.0022" y2="-22.7828" width="0.8128" layer="1"/>
-<wire x1="-35.0022" y1="-22.7828" x2="-29.0852" y2="-22.7828" width="0.8128" layer="1"/>
+<wire x1="-41.6278" y1="-5.969" x2="-41.5008" y2="-6.096" width="1.016" layer="1"/>
+<wire x1="-41.5008" y1="-6.096" x2="-34.4424" y2="-6.096" width="1.016" layer="1"/>
+<wire x1="-34.4424" y1="-6.096" x2="-33.147" y2="-7.3914" width="1.016" layer="1"/>
+<wire x1="-33.147" y1="-7.3914" x2="-33.147" y2="-20.0406" width="1.016" layer="1"/>
+<wire x1="-33.147" y1="-20.0406" x2="-30.4048" y2="-22.7828" width="1.016" layer="1"/>
+<wire x1="-30.4048" y1="-22.7828" x2="-29.0852" y2="-22.7828" width="1.016" layer="1"/>
 </signal>
 <signal name="N$4">
