File: brd/Jay_brd/Aquarius.sch (EAGLE design)
At the start: 39 parts, among them IC1 74123D, J2 DS18B20, J4 GSM/GPS, SW2 Modes, U1 DHT22, U2 DS3231SN, X1 Conn BNC : pH, X2 Conn BNC : Dissolved Oxygen, X3 Conn BNC : Conductivity, X4 Batt.1, X5 Batt.2

Commit message: Mise a jour du PCB version Jay_brd pour finalisation
Parts:
- added JP1: (no value), jumper:JP2E
- added JP2: (no value), pinhead:PINHD-1X2
- added LED1: (no value), led:LEDCHIP-LED0805
- added Q1, Q2, Q3: BSS138, m-pad-2.1:BSS138
- added R10, R12, R13, R16, R17, R18: 10K, adafruit:R-US_R0805
- added R19: 200, adafruit:R-US_R0805
- C1: device rcl:CPOL-US140CLH-0810 -> rcl:CPOL-USD
- C3: device rcl:CPOL-US140CLH-0810 -> rcl:CPOL-USB
- C4: device rcl:CPOL-US153CLV-0405 -> rcl:CPOL-USB
- L1: device rcl:L-USL8530M -> jt-inductors:L-EU10X10-EPCOS
Connections:
- new net N$1: J4.4, Q3.D, R18.1
- new net N$22: J4.3, Q2.D, R16.1
- new net N$23: J4.2, Q1.D, R12.1
- new net N$25: JP1.2, R12.2, R16.2, R18.2
- new net N$26: LED1.A, R19.1
- new net N$27: R19.2, U$1.GPIO1_16
- net 5V: now also JP1.3
- net GND: now also LED1.C
- net I2C2_SCL: now also JP2.1
- net I2C2_SDA: now also JP2.2
- net P: now also Q3.S, R17.1; no longer J4.4
- net RX: now also Q2.S, R13.1; no longer J4.3
- net TX: now also Q1.S, R10.1; no longer J4.2
- net VCC: now also JP1.1, Q1.G, Q2.G, Q3.G, R10.2, R13.2, R17.2
Other:
- moved on the sheet: J4

Commit message: Finalisation du pcb avant le test 4pcb
Parts:
- JP2: value (none) -> I2C
Changed lines of the file:
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@@
 <part name="LED1" library="led" deviceset="LED" device="CHIP-LED0805"/>
 <part name="R19" library="adafruit" deviceset="R-US_" device="R0805" value="200"/>
-<part name="JP2" library="pinhead" deviceset="PINHD-1X2" device=""/>
+<part name="JP2" library="pinhead" deviceset="PINHD-1X2" device="" value="I2C"/>
 </parts>
 <sheets>
