File: brd/Jay_brd/Aquarius.sch (EAGLE design)
At the start: 52 parts, among them IC1 74123D, J2 DS18B20, J4 GSM/GPS, Q1 BSS138, Q2 BSS138, Q3 BSS138, SW2 Modes, U1 DHT22, U2 DS3231SN, X1 Conn BNC : pH, X2 Conn BNC : Dissolved Oxygen, X3 Conn BNC : Conductivity, X4 Batt.1, X5 Batt.2

Commit message: Ajout du board V2
Other:
- note added: "Should be SDA on TX and SCL on RX"
Changed lines of the file:
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@@
 <setting verticaltext="up"/>
 </settings>
-<grid distance="0.05" unitdist="inch" unit="inch" style="lines" multiple="1" display="no" altdistance="0.01" altunitdist="inch" altunit="inch"/>
+<grid distance="0.1" unitdist="inch" unit="inch" style="lines" multiple="1" display="no" altdistance="0.01" altunitdist="inch" altunit="inch"/>
 <layers>
 <layer number="1" name="Top" color="4" fill="1" visible="no" active="no"/>
@@
 <text x="176.53" y="-68.58" size="1.778" layer="91">Vcc</text>
 <text x="176.53" y="-78.74" size="1.778" layer="91">Gnd</text>
+<text x="101.6" y="30.48" size="1.778" layer="91">Should be SDA on TX and SCL on RX</text>
 </plain>
 <instances>
