File: brd/Jay_brd V2/Aquarius.sch (EAGLE design)
At the start: 51 parts, among them IC1 74123D, J2 DS18B20, J4 GSM/GPS, Q1 BSS138, Q2 BSS138, Q3 BSS138, SW2 Modes, U1 DHT22, U2 DS3231SN, X1 Conn BNC : pH, X2 Conn BNC : Dissolved Oxygen, X3 Conn BNC : Conductivity, X4 Batt.1, X5 Batt.2

Commit message: Ajout du board V2
Parts:
- added JP2: I2C, pinhead:PINHD-1X2
- C3: device rcl:CPOL-USD -> rcl:CPOL-USB
- C4: device rcl:CPOL-US153CLV-0405 -> rcl:CPOL-USB
- L1: device rcl:L-USL8530M -> jt-inductors:L-EU10X10-EPCOS
Connections:
- new net N$28: U$1.I2C2_SDA
- net I2C2_SCL: now also JP2.1, R6.1, U$2.RX, U$3.RX, U$4.RX; no longer R5.1, U$2.TX, U$3.TX, U$4.TX
- net I2C2_SDA: now also JP2.2, R5.1, U$2.TX, U$3.TX, U$4.TX; no longer R6.1, U$1.I2C2_SDA, U$2.RX, U$3.RX, U$4.RX
